File: keyboard.kicad_pcb (KiCad board)
At the start: 2 copper layers, 189 parts, among them J1 USB_C_Receptacle_USB2.0, J10 USB_C_Receptacle_USB2.0, J11 USB_C_Receptacle_USB2.0, J2 Conn_01x02, J3 Conn_01x02, J4 Conn_01x02, J5 Conn_01x02, J6 Conn_01x03, J7 Conn_01x03, J8 Conn_01x05, J9 Conn_01x05, SW1 MXSwitch, SW10 MXSwitch, SW11 MXSwitch, SW12 MXSwitch, SW13 MXSwitch, SW14 MXSwitch, SW15 MXSwitch, SW16 MXSwitch, SW17 MXSwitch, SW18 MXSwitch, SW19 MXSwitch, SW2 MXSwitch, SW20 MXSwitch, SW21 MXSwitch, SW22 MXSwitch, SW23 MXSwitch, SW24 MXSwitch, SW25 MXSwitch, SW26 MXSwitch, SW27 MXSwitch, SW28 MXSwitch, SW29 MXSwitch, SW3 MXSwitch, SW30 MXSwitch, SW31 MXSwitch, SW32 MXSwitch, SW33 MXSwitch, SW34 MXSwitch, SW35 MXSwitch, SW36 MXSwitch, SW37 MXSwitch, SW38 MXSwitch, SW39 MXSwitch, SW4 MXSwitch, SW40 MXSwitch, SW41 MXSwitch, SW42 MXSwitch, SW43 MXSwitch, SW44 MXSwitch, SW45 MXSwitch, SW46 MXSwitch, SW47 MXSwitch, SW48 MXSwitch, SW49 MXSwitch, SW5 MXSwitch, SW50 MXSwitch, SW51 MXSwitch, SW52 MXSwitch, SW53 MXSwitch, SW54 MXSwitch, SW55 MXSwitch, SW56 MXSwitch, SW57 MXSwitch, SW58 MXSwitch, SW59 MXSwitch, SW6 MXSwitch, SW60 MXSwitch, SW61 MXSwitch, SW62 MXSwitch, SW63 MXSwitch, SW64 MXSwitch, SW65 MXSwitch, SW66 MXSwitch, SW67 MXSwitch, SW68 MXSwitch, SW69 MXSwitch, SW7 MXSwitch, SW70 MXSwitch, SW71 MXSwitch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

Commit message: Update schematics and connect pcb
Parts:
- removed J10, J11: USB_C_Receptacle_USB2.0, Connector_USB:USB_C_Receptacle_Amphenol_12401548E4-2A
- removed J7: Conn_01x03, Connector_PinHeader_2.54mm:PinHeader_1x03_P2.54mm_Vertical
- removed J8, J9: Conn_01x05, Connector_PinHeader_2.54mm:PinHeader_1x05_P2.54mm_Vertical
- removed U3, U4: AMS1117-3.3, Package_TO_SOT_SMD:SOT-223-3_TabPin2
- added C10: 10u, Capacitor_SMD:C_0201_0603Metric, B.Cu at (335.5, 23.1)
- added C11: 22pF, Capacitor_SMD:C_0201_0603Metric, B.Cu at (65.0, 23.6)
- added C12: 22pF, Capacitor_SMD:C_0201_0603Metric, B.Cu at (315.5, 23.9)
- added C13: 22pF, Capacitor_SMD:C_0201_0603Metric, B.Cu at (65.8, 23.6)
- added C14: 22pF, Capacitor_SMD:C_0201_0603Metric, B.Cu at (316.2, 23.9)
- added C15: 1uF, Capacitor_SMD:C_0201_0603Metric, B.Cu at (57.0, 10.4)
- added C16: 1uF, Capacitor_SMD:C_0201_0603Metric, B.Cu at (305.1, 10.4)
- added C5: 1u, Capacitor_SMD:C_0201_0603Metric, B.Cu at (50.0, 21.3)
- added C6: 1u, Capacitor_SMD:C_0201_0603Metric, B.Cu at (331.5, 23.1)
- added C7: 100n, Capacitor_SMD:C_0201_0603Metric, B.Cu at (332.5, 23.1)
- added C8: 100n, Capacitor_SMD:C_0201_0603Metric, B.Cu at (333.5, 23.1)
- added C9: 1u, Capacitor_SMD:C_0201_0603Metric, B.Cu at (334.5, 23.1)
- added R11: 10k, Resistor_SMD:R_0603_1608Metric, B.Cu at (71.6, 23.1)
- added R12: 10k, Resistor_SMD:R_0603_1608Metric, B.Cu at (322.3, 20.0)
- added R13: 5.1k, Resistor_SMD:R_0603_1608Metric, B.Cu at (144.3, 17.0)
- added R14: 5.1k, Resistor_SMD:R_0603_1608Metric, B.Cu at (230.9, 20.8)
- added R15: 5.1k, Resistor_SMD:R_0603_1608Metric, B.Cu at (143.5, 23.4)
- added R16: 5.1k, Resistor_SMD:R_0603_1608Metric, B.Cu at (231.4, 14.2)
- added R17: 22, Resistor_SMD:R_0603_1608Metric, B.Cu at (143.5, 19.8)
- added R18: 22, Resistor_SMD:R_0603_1608Metric, B.Cu at (231.6, 18.3)
- added R19: 22, Resistor_SMD:R_0603_1608Metric, B.Cu at (142.0, 16.3)
- added R20: 22, Resistor_SMD:R_0603_1608Metric, B.Cu at (233.2, 21.6)
- added Y1: 16MHz, Crystal:Crystal_SMD_5032-2Pin_5.0x3.2mm, B.Cu at (68.1, 21.3)
- added Y2: 16MHz, Crystal:Crystal_SMD_5032-2Pin_5.0x3.2mm, B.Cu at (318.5, 21.6)
- C1: value 10uF -> 10u
- C2: value 10uF -> 1u
- C3, C4: value 10uF -> 100n
- J2, J5: value Conn_01x02 -> USB_C_Receptacle_USB2.0; footprint Connector_PinHeader_2.54mm:PinHeader_1x02_P2.54mm_Vertical -> Connector_USB:USB_C_Receptacle_Amphenol_12401548E4-2A
- J6: value Conn_01x03 -> USB_C_Receptacle_USB2.0; footprint Connector_PinHeader_2.54mm:PinHeader_1x03_P2.54mm_Vertical -> Connector_USB:USB_C_Receptacle_Amphenol_12401548E4-2A
- R10, R9: value 5.1k -> 1k
- R5, R6, R7, R8: value 5.1k -> 22
- U1, U2: value STM32F072C8T6 -> ATmega32U4-AU; footprint Package_QFP:LQFP-48_7x7mm_P0.5mm -> Package_QFP:TQFP-44_10x10mm_P0.8mm
- moved R2 304.4 mm to (338.3, 16.8), turned to 270 degrees
- moved J2 297.5 mm to (345.2, 18.8), turned to 270 degrees
- moved J4 257.1 mm to (325.1, 20.3), turned to 180 degrees
- moved C3 191.6 mm to (41.9, 14.7), turned to 90 degrees
- moved C4 190.7 mm to (42.9, 14.7), turned to 90 degrees
- moved J3 171.8 mm to (74.2, 20.3), turned to 180 degrees
- moved J6 162.4 mm to (223.8, 18.8)
- moved R8 105.1 mm to (336.0, 16.0), turned to 0 degrees
- moved R7 104.7 mm to (38.9, 20.6), turned to 180 degrees
- moved J5 98.9 mm to (151.1, 18.8), turned to 270 degrees
- moved R4 91.8 mm to (337.8, 23.4), turned to 0 degrees
- moved R9 91.0 mm to (52.6, 25.4), turned to 0 degrees
- moved R6 86.2 mm to (336.0, 19.1), turned to 0 degrees
- moved U1 75.7 mm to (57.4, 17.8), turned to 270 degrees
- moved R10 67.0 mm to (297.9, 21.8)
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Connections:
- C2 pad 1: +3V3 -> +5V
- C4 pad 1: +3V3 -> +5V
- D10 pad 1: ROW1 -> ROW11
- D11 pad 1: ROW1 -> ROW11
- D12 pad 1: ROW1 -> ROW11
- D13 pad 1: ROW1 -> ROW11
- D14 pad 1: ROW1 -> ROW11
- D22 pad 1: ROW2 -> ROW12
- D23 pad 1: ROW2 -> ROW12
- D24 pad 1: ROW2 -> ROW12
- D25 pad 1: ROW2 -> ROW12
- D26 pad 1: ROW2 -> ROW12
- D27 pad 1: ROW2 -> ROW12
- D28 pad 1: ROW2 -> ROW12
- D36 pad 1: ROW3 -> ROW13
- D37 pad 1: ROW3 -> ROW13
- D38 pad 1: ROW3 -> ROW13
- D39 pad 1: ROW3 -> ROW13
- D40 pad 1: ROW3 -> ROW13
- D41 pad 1: ROW3 -> ROW13
- D42 pad 1: ROW3 -> ROW13
- D50 pad 1: ROW4 -> ROW14
- D51 pad 1: ROW4 -> ROW14
- D52 pad 1: ROW4 -> ROW14
- D53 pad 1: ROW4 -> ROW14
- D54 pad 1: ROW4 -> ROW14
- D55 pad 1: ROW4 -> ROW14
- D63 pad 1: ROW5 -> ROW15
- D64 pad 1: ROW5 -> ROW15
- D65 pad 1: ROW5 -> ROW15
- D66 pad 1: ROW5 -> ROW15
- D67 pad 1: ROW5 -> ROW15
- D68 pad 1: ROW5 -> ROW15
- D69 pad 1: ROW5 -> ROW15
- D75 pad 1: ROW6 -> ROW16
- D76 pad 1: ROW6 -> ROW16
- D77 pad 1: ROW6 -> ROW16
- D78 pad 1: ROW6 -> ROW16
- D79 pad 1: ROW6 -> ROW16
- D8 pad 1: ROW1 -> ROW11
- D80 pad 1: ROW6 -> ROW16
- D9 pad 1: ROW1 -> ROW11
- J1 pad A6: D_P -> Net-(J1-PadA6)
- J1 pad A7: D_N -> Net-(J1-PadA7)
- J1 pad B6: D_P -> Net-(J1-PadA6)
- J1 pad B7: D_N -> Net-(J1-PadA7)
- J3 pad 1: RESET1 -> RESET0
- J4 pad 1: +3V3 -> RESET1
- J4 pad 2: BOOT0 -> GND
- R10 pad 2: Net-(J11-PadB5) -> Net-(R10-Pad2)
- R2 pad 2: Net-(J1-PadB5) -> Net-(J2-PadA5)
- R3 pad 1: RESET0 -> GND
- R3 pad 2: +3V3 -> Net-(J1-PadB5)
- R4 pad 1: RESET1 -> GND
- R4 pad 2: +3V3 -> Net-(J2-PadB5)
- R5 pad 1: BOOT0 -> D_NJ1
- R5 pad 2: GND -> Net-(J1-PadA7)
- R6 pad 1: BOOT1 -> D_NJ2
- R6 pad 2: GND -> Net-(J2-PadA7)
- R7 pad 1: GND -> D_PJ1
- R7 pad 2: Net-(J10-PadA5) -> Net-(J1-PadA6)
- R8 pad 1: GND -> D_PJ2
- R8 pad 2: Net-(J11-PadA5) -> Net-(J2-PadA6)
- R9 pad 2: Net-(J10-PadB5) -> Net-(R9-Pad2)
- U1 pad 1: +3V3 -> Net-(U1-Pad1)
- U1 pad 10: ROW01 -> D_PJ5
- U1 pad 11: ROW02 -> D_NJ5
- U1 pad 12: ROW03 -> Net-(U1-Pad12)
- U1 pad 13: ROW04 -> RESET0
- U1 pad 14: ROW05 -> +5V
- U1 pad 15: ROW06 -> GND
- U1 pad 17: D_NJ2 -> Net-(C11-Pad1)
- U1 pad 18: COL01 -> Net-(U1-Pad18)
- U1 pad 19: COL02 -> Net-(U1-Pad19)
- U1 pad 2: Net-(U1-Pad2) -> +5V
- U1 pad 20: COL03 -> Net-(U1-Pad20)
- U1 pad 24: +3V3 -> +5V
- U1 pad 26: Net-(U1-Pad26) -> COL07
- U1 pad 27: Net-(U1-Pad27) -> COL06
- U1 pad 28: Net-(U1-Pad28) -> COL05
- U1 pad 29: D_PJ2 -> COL04
- U1 pad 3: Net-(U1-Pad3) -> D_NJ1
- U1 pad 30: PA09 -> COL03
- U1 pad 31: Net-(U1-Pad31) -> COL02
- U1 pad 32: D_N -> COL01
- U1 pad 33: D_P -> Net-(R9-Pad2)
- U1 pad 34: SWDIO0 -> +5V
- U1 pad 36: +3V3 -> ROW01
- U1 pad 37: SWCLK0 -> ROW02
- U1 pad 38: Net-(U1-Pad38) -> ROW03
- U1 pad 39: COL04 -> ROW04
- U1 pad 4: Net-(U1-Pad4) -> D_PJ1
- U1 pad 40: COL05 -> ROW05
- U1 pad 41: COL06 -> ROW06
- U1 pad 42: COL07 -> +5V
- U1 pad 43: Net-(U1-Pad43) -> GND
- U1 pad 44: BOOT0 -> +5V
- U1 pad 5: Net-(U1-Pad5) -> GND
- U1 pad 7: RESET0 -> +5V
- U1 pad 8: GND -> Net-(U1-Pad8)
- U1 pad 9: +3V3 -> Net-(U1-Pad9)
- U2 pad 1: +3V3 -> Net-(U2-Pad1)
- U2 pad 10: ROW11 -> D_NJ6
- U2 pad 11: ROW12 -> D_PJ6
- U2 pad 12: ROW13 -> Net-(U2-Pad12)
- U2 pad 13: ROW14 -> RESET1
- U2 pad 14: ROW15 -> +5V
- U2 pad 15: ROW16 -> GND
- U2 pad 17: D_NJ3 -> Net-(C12-Pad1)
- U2 pad 18: COL08 -> Net-(U2-Pad18)
- U2 pad 19: COL09 -> Net-(U2-Pad19)
- U2 pad 2: Net-(U2-Pad2) -> +5V
- U2 pad 20: COL10 -> Net-(U2-Pad20)
- U2 pad 24: +3V3 -> +5V
- U2 pad 26: Net-(U2-Pad26) -> COL14
- U2 pad 27: Net-(U2-Pad27) -> COL13
- U2 pad 28: Net-(U2-Pad28) -> COL12
- U2 pad 29: D_PJ3 -> COL11
- U2 pad 3: Net-(U2-Pad3) -> D_NJ2
- U2 pad 30: PA19 -> COL10
- U2 pad 31: Net-(U2-Pad31) -> COL09
- U2 pad 32: Net-(U2-Pad32) -> COL08
- U2 pad 33: Net-(U2-Pad33) -> Net-(R10-Pad2)
- U2 pad 34: SWDIO1 -> +5V
- U2 pad 36: +3V3 -> ROW11
- U2 pad 37: SWCLK1 -> ROW12
- U2 pad 38: Net-(U2-Pad38) -> ROW13
- U2 pad 39: COL11 -> ROW14
- U2 pad 4: Net-(U2-Pad4) -> D_PJ2
- U2 pad 40: COL12 -> ROW15
- U2 pad 41: COL13 -> ROW16
- U2 pad 42: COL14 -> +5V
- U2 pad 43: Net-(U2-Pad43) -> GND
- U2 pad 44: BOOT1 -> +5V
- U2 pad 5: Net-(U2-Pad5) -> GND
- U2 pad 7: RESET1 -> +5V
- U2 pad 8: GND -> Net-(U2-Pad8)
- U2 pad 9: +3V3 -> Net-(U2-Pad9)
Routing:
- net GND: track 57.8 -> 428.8 mm, vias 0 -> 7
- net +5V: track 18.1 -> 342.1 mm, vias 0 -> 11
- net ROW16: track 0.00 -> 288.2 mm
- net ROW15: track 0.00 -> 275.4 mm
- net ROW14: track 0.00 -> 247.3 mm
- net ROW13: track 0.00 -> 235.3 mm
- net ROW12: track 0.00 -> 215.2 mm
- net ROW06: track 86.9 -> 214.3 mm
- net ROW11: track 0.00 -> 126.2 mm
- net ROW5: track 114.0 -> 0.00 mm
- net ROW3: track 114.0 -> 0.00 mm
- net ROW2: track 114.0 -> 0.00 mm
- net ROW1: track 114.0 -> 0.00 mm
- net ROW05: track 114.0 -> 221.3 mm
- net ROW4: track 105.9 -> 0.00 mm
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Other:
- board outline added: 329.7 x 130 mm

Commit message: Update sch and added qmk files
Parts:
- removed R13, R14, R15, R16: 5.1k, Resistor_SMD:R_0603_1608Metric
- moved R19 3.81 mm to (144.3, 13.2)
- moved R20 2.65 mm to (230.6, 22.4)
- moved R17 1.93 mm to (144.3, 18.0)
- moved C10 1.83 mm to (337.1, 22.1)
- moved C6 1.83 mm to (333.0, 22.1)
- moved C7 1.83 mm to (334.0, 22.1)
- moved C8 1.83 mm to (335.0, 22.1)
- moved C9 1.83 mm to (336.0, 22.1)
- moved R6 1.83 mm to (337.6, 18.0)
- moved R2 1.83 mm to (339.9, 15.7)
- moved J2 1.83 mm to (346.7, 17.8)
- moved R4 1.83 mm to (339.3, 22.4)
- moved R8 1.83 mm to (337.6, 15.0)
- moved C1 1.52 mm to (38.4, 14.7)
- moved C2 1.52 mm to (39.4, 14.7)
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Routing:
- net Net-(J6-PadB5): track 9.29 -> 0.00 mm
- net Net-(J5-PadB5): track 9.11 -> 0.00 mm
- net GND: track 428.8 -> 425.8 mm
- net +5V: track 342.1 -> 344.9 mm
- net D_PJ6: track 83.7 -> 86.6 mm
- net Net-(J6-PadA5): track 2.28 -> 0.00 mm
- net Net-(J6-PadA6): track 18.7 -> 16.5 mm
- net Net-(J5-PadA5): track 1.92 -> 0.00 mm
- net Net-(J5-PadA6): track 18.4 -> 16.5 mm
- net D_PJ1: track 25.6 -> 27.1 mm
- net D_NJ1: track 21.7 -> 23.2 mm
- net D_NJ6: track 91.2 -> 92.5 mm
- net D_PJ2: track 34.2 -> 35.3 mm
- net D_NJ2: track 37.2 -> 38.3 mm
- net D_PJ5: track 83.9 -> 85.0 mm

Commit message: Updates
Parts:
- moved R9 1.52 mm to (51.1, 25.4)
- renumbered R17 to R13, R18 to R14, R19 to R15, R20 to R16
Connections:
- U1 pad 10: D_PJ5 -> Net-(U1-Pad10)
- U1 pad 11: D_NJ5 -> Net-(U1-Pad11)
- U1 pad 18: Net-(U1-Pad18) -> D_PJ5
- U1 pad 19: Net-(U1-Pad19) -> D_NJ5
- U2 pad 10: D_NJ6 -> Net-(U2-Pad10)
- U2 pad 11: D_PJ6 -> Net-(U2-Pad11)
- U2 pad 18: Net-(U2-Pad18) -> D_NJ6
- U2 pad 19: Net-(U2-Pad19) -> D_PJ6
Routing:
- net D_NJ6: track 92.5 -> 88.8 mm
- net D_PJ5: track 85.0 -> 82.8 mm, vias 0 -> 2
- net COL03: track 117.1 -> 118.6 mm
- net D_NJ5: track 84.8 -> 83.7 mm, vias 0 -> 2
- net COL04: track 135.1 -> 136.0 mm
- net D_PJ6: track 86.6 -> 85.7 mm
- net COL02: track 100.6 -> 101.5 mm
- net Net-(R9-Pad2): track 1.92 -> 2.55 mm
- net GND: track 425.8 -> 425.2 mm
- net COL12: track 100.7 -> 101.3 mm
- net COL05: track 157.0 -> 157.6 mm
