File: keyboard.sch (KiCad schematic (older format))
At the start: 189 parts, among them J1 USB_C_Receptacle_USB2.0, J10 USB_C_Receptacle_USB2.0, J11 USB_C_Receptacle_USB2.0, J2 Conn_01x02, J3 Conn_01x02, J4 Conn_01x02, J5 Conn_01x02, J6 Conn_01x03, J7 Conn_01x03, J8 Conn_01x05, J9 Conn_01x05, SW1 MXSwitch, SW10 MXSwitch, SW11 MXSwitch, SW12 MXSwitch, SW13 MXSwitch, SW14 MXSwitch, SW15 MXSwitch, SW16 MXSwitch, SW17 MXSwitch, SW18 MXSwitch, SW19 MXSwitch, SW2 MXSwitch, SW20 MXSwitch, SW21 MXSwitch, SW22 MXSwitch, SW23 MXSwitch, SW24 MXSwitch, SW25 MXSwitch, SW26 MXSwitch, SW27 MXSwitch, SW28 MXSwitch, SW29 MXSwitch, SW3 MXSwitch, SW30 MXSwitch, SW31 MXSwitch, SW32 MXSwitch, SW33 MXSwitch, SW34 MXSwitch, SW35 MXSwitch, SW36 MXSwitch, SW37 MXSwitch, SW38 MXSwitch, SW39 MXSwitch, SW4 MXSwitch, SW40 MXSwitch, SW41 MXSwitch, SW42 MXSwitch, SW43 MXSwitch, SW44 MXSwitch, SW45 MXSwitch, SW46 MXSwitch, SW47 MXSwitch, SW48 MXSwitch, SW49 MXSwitch, SW5 MXSwitch, SW50 MXSwitch, SW51 MXSwitch, SW52 MXSwitch, SW53 MXSwitch, SW54 MXSwitch, SW55 MXSwitch, SW56 MXSwitch, SW57 MXSwitch, SW58 MXSwitch, SW59 MXSwitch, SW6 MXSwitch, SW60 MXSwitch, SW61 MXSwitch, SW62 MXSwitch, SW63 MXSwitch, SW64 MXSwitch, SW65 MXSwitch, SW66 MXSwitch, SW67 MXSwitch, SW68 MXSwitch, SW69 MXSwitch, SW7 MXSwitch, SW70 MXSwitch, SW71 MXSwitch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

Commit message: Update schematics and connect pcb
Parts:
- removed C1, C2, C3, C4: 10uF, Capacitor_SMD:C_0201_0603Metric, symbol Device:C
- removed J10, J11: USB_C_Receptacle_USB2.0, Connector_USB:USB_C_Receptacle_Amphenol_12401548E4-2A, symbol Connector:USB_C_Receptacle_USB2.0
- removed J2, J5: Conn_01x02, Connector_PinHeader_2.54mm:PinHeader_1x02_P2.54mm_Vertical, symbol Connector_Generic:Conn_01x02
- removed J6, J7: Conn_01x03, Connector_PinHeader_2.54mm:PinHeader_1x03_P2.54mm_Vertical, symbol Connector_Generic:Conn_01x03
- removed J8, J9: Conn_01x05, Connector_PinHeader_2.54mm:PinHeader_1x05_P2.54mm_Vertical, symbol Connector_Generic:Conn_01x05
- removed R1, R10, R2, R3, R4, R5, R6, R7, R8, R9: 5.1k, Resistor_SMD:R_0603_1608Metric, symbol Device:R
- removed U1, U2: STM32F072C8T6, Package_QFP:LQFP-48_7x7mm_P0.5mm, symbol MCU_ST_STM32F0:STM32F072C8Tx
- removed U3, U4: AMS1117-3.3, Package_TO_SOT_SMD:SOT-223-3_TabPin2, symbol Regulator_Linear:AMS1117-3.3
- added C1, C10: 10u, Capacitor_SMD:C_0201_0603Metric, symbol Device:C_Small
- added C11, C12, C13, C14: 22pF, Capacitor_SMD:C_0201_0603Metric, symbol Device:C_Small
- added C15, C16: 1uF, Capacitor_SMD:C_0201_0603Metric, symbol Device:C_Small
- added C2, C5, C6, C9: 1u, Capacitor_SMD:C_0201_0603Metric, symbol Device:C_Small
- added C3, C4, C7, C8: 100n, Capacitor_SMD:C_0201_0603Metric, symbol Device:C_Small
- added J2, J5, J6: USB_C_Receptacle_USB2.0, Connector_USB:USB_C_Receptacle_Amphenol_12401548E4-2A, symbol Connector:USB_C_Receptacle_USB2.0
- added R1, R13, R14, R15, R16, R2, R3, R4: 5.1k, Resistor_SMD:R_0603_1608Metric, symbol Device:R_Small
- added R10, R9: 1k, Resistor_SMD:R_0603_1608Metric, symbol Device:R_Small
- added R11, R12: 10k, Resistor_SMD:R_0603_1608Metric, symbol Device:R_Small
- added R17, R18, R19, R20, R5, R6, R7, R8: 22, Resistor_SMD:R_0603_1608Metric, symbol Device:R_Small
- added U1, U2: ATmega32U4-AU, Package_QFP:TQFP-44_10x10mm_P0.8mm, symbol MCU_Microchip_ATmega:ATmega32U4-AU
- added Y1, Y2: 16MHz, Crystal:Crystal_SMD_5032-2Pin_5.0x3.2mm, symbol Device:Crystal_Small
Connections:
- net +3V3 is gone; now on net RESET1: J4.1 (Pin_1)
- net BOOT0 is gone; now on net GND: J4.2 (Pin_2)
- net ROW1 is gone; now on net ROW11: D10.1 (K), D11.1 (K), D12.1 (K), D13.1 (K), D14.1 (K), D8.1 (K), D9.1 (K)
- net ROW2 is gone; now on net ROW12: D22.1 (K), D23.1 (K), D24.1 (K), D25.1 (K), D26.1 (K), D27.1 (K), D28.1 (K)
- net ROW3 is gone; now on net ROW13: D36.1 (K), D37.1 (K), D38.1 (K), D39.1 (K), D40.1 (K), D41.1 (K), D42.1 (K)
- net ROW4 is gone; now on net ROW14: D50.1 (K), D51.1 (K), D52.1 (K), D53.1 (K), D54.1 (K), D55.1 (K)
- net ROW5 is gone; now on net ROW15: D63.1 (K), D64.1 (K), D65.1 (K), D66.1 (K), D67.1 (K), D68.1 (K), D69.1 (K)
- net ROW6 is gone; now on net ROW16: D75.1 (K), D76.1 (K), D77.1 (K), D78.1 (K), D79.1 (K), D80.1 (K)
- net +5V: now also C1.1, C10.1, C2.1, C3.1, C4.1, C5.1, C6.1, C7.1, C8.1, C9.1, J2.A4 (VBUS), J2.A9 (VBUS), J2.B4 (VBUS), J2.B9 (VBUS), J5.A4 (VBUS), J5.A9 (VBUS), J5.B4 (VBUS), J5.B9 (VBUS), J6.A4 (VBUS), J6.A9 (VBUS), J6.B4 (VBUS), J6.B9 (VBUS), R11.1, R12.1, U1.14 (VCC), U1.2 (UVCC), U1.24 (AVCC), U1.34 (VCC), U1.42 (AREF), U1.44 (AVCC), U1.7 (VBUS), U2.14 (VCC), U2.2 (UVCC), U2.24 (AVCC), U2.34 (VCC), U2.42 (AREF), U2.44 (AVCC), U2.7 (VBUS)
- net COL01: now also U1.32 (PC7)
- net COL02: now also U1.31 (PC6)
- net COL03: now also U1.30 (PB6)
- net COL04: now also U1.29 (PB5)
- net COL05: now also U1.28 (PB4)
- net COL06: now also U1.27 (PD7)
- net COL07: now also U1.26 (PD6)
- net COL08: now also U2.32 (PC7)
- net COL09: now also U2.31 (PC6)
- net COL10: now also U2.30 (PB6)
- net COL11: now also U2.29 (PB5)
- net COL12: now also U2.28 (PB4)
- net COL13: now also U2.27 (PD7)
- net COL14: now also U2.26 (PD6)
- net D_NJ2: now also R6.1, U2.3 (D-)
- net D_PJ2: now also R8.1, U2.4 (D+)
- net GND: now also C1.2, C10.2, C11.2, C12.2, C13.1, C14.1, C15.1, C16.1, C2.2, C3.2, C4.2, C5.2, C6.2, C7.2, C8.2, C9.2, J2.A1 (GND), J2.A12 (GND), J2.B1 (GND), J2.B12 (GND), J2.S1 (SHIELD), J5.A1 (GND), J5.A12 (GND), J5.B1 (GND), J5.B12 (GND), J5.S1 (SHIELD), J6.A1 (GND), J6.A12 (GND), J6.B1 (GND), J6.B12 (GND), J6.S1 (SHIELD), R1.1, R10.1, R13.1, R14.1, R15.1, R16.1, R2.1, R3.1, R4.1, R9.1, U1.15 (GND), U1.23 (GND), U1.35 (GND), U1.43 (GND), U1.5 (UGND), U2.15 (GND), U2.23 (GND), U2.35 (GND), U2.43 (GND), U2.5 (UGND)
- net RESET0: now also J3.1 (Pin_1), R11.2, U1.13 (~RESET)
- net RESET1: now also R12.2, U2.13 (~RESET); no longer J3.1 (Pin_1)
- net ROW01: now also U1.36 (PF7)
- net ROW02: now also U1.37 (PF6)
- net ROW03: now also U1.38 (PF5)
- net ROW04: now also U1.39 (PF4)
- net ROW05: now also U1.40 (PF1)
- net ROW06: now also U1.41 (PF0)
- net ROW11: now also U2.36 (PF7)
- net ROW12: now also U2.37 (PF6)
- net ROW13: now also U2.38 (PF5)
- net ROW14: now also U2.39 (PF4)
- net ROW15: now also U2.40 (PF1)
- net ROW16: now also U2.41 (PF0)
- net at J1.A5 (CC1): now also R1.2
- net at J1.B5 (CC2): now also R3.2
- net D_N: no longer names the net of J1.A7 (D-), J1.B7 (D-)
- net D_N: now also R5.2
- net D_P: no longer names the net of J1.A6 (D+), J1.B6 (D+)
- net D_P: now also R7.2
- new net: C13.2, U1.16 (XTAL2), Y1.2
- new net: C11.1, U1.17 (XTAL1), Y1.1
- new net: R9.2, U1.33 (~HWB~/PE2)
- new net: C15.2, U1.6 (UCAP)
- new net: J5.A5 (CC1), R13.2
- new net: J5.A6 (D+), J5.B6 (D+), R19.2
- new net: J5.A7 (D-), J5.B7 (D-), R17.2
- new net: J5.B5 (CC2), R15.2
- new net: J2.A5 (CC1), R2.2
- new net: J2.A6 (D+), J2.B6 (D+), R8.2
- new net: J2.A7 (D-), J2.B7 (D-), R6.2
- new net: J2.B5 (CC2), R4.2
- new net: C14.2, U2.16 (XTAL2), Y2.2
- new net: C12.1, U2.17 (XTAL1), Y2.1
- new net: R10.2, U2.33 (~HWB~/PE2)
- new net: C16.2, U2.6 (UCAP)
- new net: J6.A5 (CC1), R14.2
- new net: J6.A6 (D+), J6.B6 (D+), R20.2
- new net: J6.A7 (D-), J6.B7 (D-), R18.2
- new net: J6.B5 (CC2), R16.2
- new net D_NJ1: R5.1, U1.3 (D-)
- new net D_NJ5: R17.1, U1.11 (PB3)
- new net D_NJ6: R18.1, U2.10 (PB2)
- new net D_PJ1: R7.1, U1.4 (D+)
- new net D_PJ5: R19.1, U1.10 (PB2)
- new net D_PJ6: R20.1, U2.11 (PB3)
- no-connect marks 42 -> 8

Commit message: Update sch and added qmk files
Parts:
- removed R13, R14, R15, R16: 5.1k, Resistor_SMD:R_0603_1608Metric, symbol Device:R_Small
Connections:
- net D_NJ5: now also U1.19 (PD1); no longer U1.11 (PB3)
- net D_NJ6: now also U2.18 (PD0); no longer U2.10 (PB2)
- net D_PJ5: now also U1.18 (PD0); no longer U1.10 (PB2)
- net D_PJ6: now also U2.19 (PD1); no longer U2.11 (PB3)
- no-connect marks 8 -> 32
Changed lines of the file:
@@
 Text GLabel 20650 5550 0    50   Input ~ 0
 ROW16
-Text GLabel 20650 3350 0    50   Input ~ 0
+Text GLabel 20650 4350 0    50   Input ~ 0
 D_NJ6
-Text GLabel 20650 3450 0    50   Input ~ 0
+Text GLabel 20650 4450 0    50   Input ~ 0
 D_PJ6
 Text GLabel 17450 900  2    50   Input ~ 0
@@
 	0    1    1    0
 $EndComp
-$Comp
-L power:GND #PWR031
-U 1 1 61D05F3F
-P 1800 8250
-F 0 "#PWR031" H 1800 8000 50  0001 C CNN
-F 1 "GND" V 1805 8122 50  0000 R CNN
-F 2 "" H 1800 8250 50  0001 C CNN
-F 3 "" H 1800 8250 50  0001 C CNN
-	1    1800 8250
-	0    -1   -1   0
-$EndComp
 Text GLabel 1800 8550 2    50   Input ~ 0
 D_NJ5
@@
 Wire Wire Line
 	850  9500 1000 9500
-Wire Wire Line
-	1800 8200 1800 8250
-Connection ~ 1800 8250
-Wire Wire Line
-	1800 8250 1800 8300
-$Comp
-L Device:R_Small R13
-U 1 1 61D05F64
-P 1700 8200
-F 0 "R13" V 1600 8150 50  0000 C CNN
-F 1 "5.1k" V 1600 8350 50  0000 C CNN
-F 2 "Resistor_SMD:R_0603_1608Metric" H 1700 8200 50  0001 C CNN
-F 3 "~" H 1700 8200 50  0001 C CNN
-F 4 "C14677" V 1700 8200 50  0001 C CNN "LCSC"
-	1    1700 8200
-	0    1    1    0
-$EndComp
-$Comp
-L Device:R_Small R15
-U 1 1 61D05F6B
-P 1700 8300
-F 0 "R15" V 1800 8250 50  0000 C CNN
-F 1 "5.1k" V 1800 8450 50  0000 C CNN
-F 2 "Resistor_SMD:R_0603_1608Metric" H 1700 8300 50  0001 C CNN
-F 3 "~" H 1700 8300 50  0001 C CNN
-F 4 "C14677" V 1700 8300 50  0001 C CNN "LCSC"
-	1    1700 8300
-	0    1    1    0
-$EndComp
 $Comp
 L Connector:USB_C_Receptacle_USB2.0 J2
@@
 	0    -1   1    0
 $EndComp
-$Comp
-L power:GND #PWR032
-U 1 1 61E67B14
-P 21600 8250
-F 0 "#PWR032" H 21600 8000 50  0001 C CNN
-F 1 "GND" V 21605 8122 50  0000 R CNN
-F 2 "" H 21600 8250 50  0001 C CNN
-F 3 "" H 21600 8250 50  0001 C CNN
-	1    21600 8250
-	0    1    -1   0
-$EndComp
 Text GLabel 21600 8550 0    50   Input ~ 0
 D_NJ6
@@
 Wire Wire Line
 	22550 9500 22400 9500
-Wire Wire Line
-	21600 8200 21600 8250
-Connection ~ 21600 8250
-Wire Wire Line
-	21600 8250 21600 8300
-$Comp
-L Device:R_Small R14
-U 1 1 61E67B39
-P 21700 8200
-F 0 "R14" V 21600 8150 50  0000 C CNN
-F 1 "5.1k" V 21600 8350 50  0000 C CNN
-F 2 "Resistor_SMD:R_0603_1608Metric" H 21700 8200 50  0001 C CNN
-F 3 "~" H 21700 8200 50  0001 C CNN
-F 4 "C14677" V 21700 8200 50  0001 C CNN "LCSC"
-	1    21700 8200
-	0    -1   1    0
-$EndComp
-$Comp
-L Device:R_Small R16
-U 1 1 61E67B40
-P 21700 8300
-F 0 "R16" V 21800 8250 50  0000 C CNN
-F 1 "5.1k" V 21800 8450 50  0000 C CNN
-F 2 "Resistor_SMD:R_0603_1608Metric" H 21700 8300 50  0001 C CNN
-F 3 "~" H 21700 8300 50  0001 C CNN
-F 4 "C14677" V 21700 8300 50  0001 C CNN "LCSC"
-	1    21700 8300
-	0    -1   1    0
-$EndComp
 $Comp
 L Device:C_Small C5
@@
 	0    1    1    0
 $EndComp
-Text GLabel 2700 3350 2    50   Input ~ 0
+Text GLabel 2700 4350 2    50   Input ~ 0
 D_PJ5
-Text GLabel 2700 3450 2    50   Input ~ 0
+Text GLabel 2700 4450 2    50   Input ~ 0
 D_NJ5
+NoConn ~ 1600 8200
+NoConn ~ 1600 8300
+NoConn ~ 21800 8200
+NoConn ~ 21800 8300
+NoConn ~ 2700 5350
+NoConn ~ 2700 4850
+NoConn ~ 2700 4750
+NoConn ~ 2700 4650
+NoConn ~ 2700 4550
+NoConn ~ 2700 3850
+NoConn ~ 2700 3450
+NoConn ~ 2700 3350
+NoConn ~ 2700 3250
+NoConn ~ 2700 3150
+NoConn ~ 20650 5350
+NoConn ~ 20650 4850
+NoConn ~ 20650 4750
+NoConn ~ 20650 4650
+NoConn ~ 20650 4550
+NoConn ~ 20650 3850
+NoConn ~ 20650 3450
+NoConn ~ 20650 3350
+NoConn ~ 20650 3250
+NoConn ~ 20650 3150
 $EndSCHEMATC

Commit message: Updates
Parts:
- J3, J4: LCSC (none) -> C492401
- Y1, Y2: LCSC C568455 -> C12668
- renumbered R17 to R13, R18 to R14, R19 to R15, R20 to R16
Changed lines of the file:
@@
 F 2 "Crystal:Crystal_SMD_5032-2Pin_5.0x3.2mm" H 1300 3450 50  0001 C CNN
 F 3 "~" H 1300 3450 50  0001 C CNN
-F 4 "C568455" V 1300 3450 50  0001 C CNN "LCSC"
+F 4 "C12668" V 1300 3450 50  0001 C CNN "LCSC"
 	1    1300 3450
 	0    1    1    0
@@
 F 2 "Connector_PinHeader_2.54mm:PinHeader_1x02_P2.54mm_Vertical" H 1100 7350 50  0001 C CNN
 F 3 "~" H 1100 7350 50  0001 C CNN
+F 4 "C492401" H 1100 7350 50  0001 C CNN "LCSC"
 	1    1100 7350
 	-1   0    0    -1
@@
 $EndComp
 $Comp
-L power:GND #PWR033
+L power:GND #PWR031
 U 1 1 61D05F33
 P 850 9500
-F 0 "#PWR033" H 850 9250 50  0001 C CNN
+F 0 "#PWR031" H 850 9250 50  0001 C CNN
 F 1 "GND" H 855 9327 50  0000 C CNN
 F 2 "" H 850 9500 50  0001 C CNN
@@
 	1600 8500 1600 8550
 $Comp
-L Device:R_Small R19
+L Device:R_Small R15
 U 1 1 61D05F52
 P 1700 8750
-F 0 "R19" V 1800 8700 50  0000 C CNN
+F 0 "R15" V 1800 8700 50  0000 C CNN
 F 1 "22" V 1800 8850 50  0000 C CNN
 F 2 "Resistor_SMD:R_0603_1608Metric" H 1700 8750 50  0001 C CNN
@@
 F 2 "Crystal:Crystal_SMD_5032-2Pin_5.0x3.2mm" H 22050 3450 50  0001 C CNN
 F 3 "~" H 22050 3450 50  0001 C CNN
-F 4 "C568455" V 22050 3450 50  0001 C CNN "LCSC"
+F 4 "C12668" V 22050 3450 50  0001 C CNN "LCSC"
 	1    22050 3450
 	0    -1   1    0
@@
 F 2 "Connector_PinHeader_2.54mm:PinHeader_1x02_P2.54mm_Vertical" H 22300 7350 50  0001 C CNN
 F 3 "~" H 22300 7350 50  0001 C CNN
+F 4 "C492401" H 22300 7350 50  0001 C CNN "LCSC"
 	1    22300 7350
 	1    0    0    -1
@@
 $EndComp
 $Comp
-L power:GND #PWR034
+L power:GND #PWR032
 U 1 1 61E67B08
 P 22550 9500
-F 0 "#PWR034" H 22550 9250 50  0001 C CNN
+F 0 "#PWR032" H 22550 9250 50  0001 C CNN
 F 1 "GND" H 22555 9327 50  0000 C CNN
 F 2 "" H 22550 9500 50  0001 C CNN
@@
 	21800 8500 21800 8550
 $Comp
-L Device:R_Small R18
+L Device:R_Small R14
 U 1 1 61E67B20
 P 21700 8550
-F 0 "R18" V 21800 8500 50  0000 C CNN
+F 0 "R14" V 21800 8500 50  0000 C CNN
 F 1 "22" V 21800 8650 50  0000 C CNN
 F 2 "Resistor_SMD:R_0603_1608Metric" H 21700 8550 50  0001 C CNN
@@
 $EndComp
 $Comp
-L Device:R_Small R20
+L Device:R_Small R16
 U 1 1 61E67B27
 P 21700 8750
-F 0 "R20" V 21800 8700 50  0000 C CNN
+F 0 "R16" V 21800 8700 50  0000 C CNN
 F 1 "22" V 21800 8850 50  0000 C CNN
 F 2 "Resistor_SMD:R_0603_1608Metric" H 21700 8750 50  0001 C CNN
@@
 Connection ~ 19700 1500
 $Comp
-L Device:R_Small R17
+L Device:R_Small R13
 U 1 1 61D05F4B
 P 1700 8550
-F 0 "R17" V 1800 8500 50  0000 C CNN
+F 0 "R13" V 1800 8500 50  0000 C CNN
 F 1 "22" V 1800 8650 50  0000 C CNN
 F 2 "Resistor_SMD:R_0603_1608Metric" H 1700 8550 50  0001 C CNN
